Commit message: 2018-12-28 new

File: src3/robot_description/urdf/invite_csda10f.xacro (robot description, xacro)
@@ -54,5 +54,5 @@
   <link name="camera_link"/>
    <joint name="camera_link_fix" type="fixed">
-     <origin xyz="0.0 1.09 0.57" rpy="0 ${-13*pi/18} ${pi/2}"/>
+     <origin xyz="0.05 0.9 0.55" rpy="0 ${-0.8*pi} ${pi/2}"/>
      <parent link="camera_link"/>
      <child link="base_link"/>
